File: ItsyBitsy Expander v1.0/ItsyBitsy_Expander_v1.0.sch (EAGLE design)
At the start: 45 parts, among them CN2 JSTPH, IC1 74AHC1G125, J1 H4P-SMD-2.0, J10 H4P-SMD-2.0, J11 H4P-SMD-2.0, J12 H4P-SMD-2.0, J2 H4P-SMD-2.0, J3 H4P-SMD-2.0, J4 H4P-SMD-2.0, J5 H4P-SMD-2.0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

Commit message: Fix bug in ESP32 footprint
Flip RX and TX pads
Changed lines of the file:
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@@
 <grid distance="0.1" unitdist="inch" unit="inch" style="lines" multiple="1" display="no" altdistance="0.01" altunitdist="inch" altunit="inch"/>
 <layers>
-<layer number="1" name="Top" color="4" fill="1" visible="yes" active="no"/>
-<layer number="2" name="Route2" color="16" fill="1" visible="yes" active="no"/>
-<layer number="3" name="Route3" color="17" fill="1" visible="yes" active="no"/>
-<layer number="4" name="Route4" color="18" fill="1" visible="yes" active="no"/>
-<layer number="5" name="Route5" color="19" fill="1" visible="yes" active="no"/>
-<layer number="6" name="Route6" color="25" fill="1" visible="yes" active="no"/>
-<layer number="7" name="Route7" color="26" fill="1" visible="yes" active="no"/>
-<layer number="8" name="Route8" color="27" fill="1" visible="yes" active="no"/>
-<layer number="9" name="Route9" color="28" fill="1" visible="yes" active="no"/>
-<layer number="10" name="Route10" color="29" fill="1" visible="yes" active="no"/>
-<layer number="11" name="Route11" color="30" fill="1" visible="yes" active="no"/>
-<layer number="12" name="Route12" color="20" fill="1" visible="yes" active="no"/>
-<layer number="13" name="Route13" color="21" fill="1" visible="yes" active="no"/>
-<layer number="14" name="Route14" color="22" fill="1" visible="yes" active="no"/>
-<layer number="15" name="Route15" color="23" fill="1" visible="yes" active="no"/>
-<layer number="16" name="Bottom" color="1" fill="1" visible="yes" active="no"/>
-<layer number="17" name="Pads" color="2" fill="1" visible="yes" active="no"/>
-<layer number="18" name="Vias" color="2" fill="1" visible="yes" active="no"/>
-<layer number="19" name="Unrouted" color="6" fill="1" visible="yes" active="no"/>
-<layer number="20" name="Dimension" color="24" fill="1" visible="yes" active="no"/>
-<layer number="21" name="tPlace" color="7" fill="1" visible="yes" active="no"/>
-<layer number="22" name="bPlace" color="7" fill="1" visible="yes" active="no"/>
-<layer number="23" name="tOrigins" color="15" fill="1" visible="yes" active="no"/>
-<layer number="24" name="bOrigins" color="15" fill="1" visible="yes" active="no"/>
-<layer number="25" name="tNames" color="7" fill="1" visible="yes" active="no"/>
-<layer number="26" name="bNames" color="7" fill="1" visible="yes" active="no"/>
-<layer number="27" name="tValues" color="7" fill="1" visible="yes" active="no"/>
-<layer number="28" name="bValues" color="7" fill="1" visible="yes" active="no"/>
+<layer number="1" name="Top" color="4" fill="1" visible="no" active="no"/>
+<layer number="2" name="Route2" color="16" fill="1" visible="no" active="no"/>
+<layer number="3" name="Route3" color="17" fill="1" visible="no" active="no"/>
+<layer number="4" name="Route4" color="18" fill="1" visible="no" active="no"/>
+<layer number="5" name="Route5" color="19" fill="1" visible="no" active="no"/>
+<layer number="6" name="Route6" color="25" fill="1" visible="no" active="no"/>
+<layer number="7" name="Route7" color="26" fill="1" visible="no" active="no"/>
+<layer number="8" name="Route8" color="27" fill="1" visible="no" active="no"/>
+<layer number="9" name="Route9" color="28" fill="1" visible="no" active="no"/>
+<layer number="10" name="Route10" color="29" fill="1" visible="no" active="no"/>
+<layer number="11" name="Route11" color="30" fill="1" visible="no" active="no"/>
+<layer number="12" name="Route12" color="20" fill="1" visible="no" active="no"/>
+<layer number="13" name="Route13" color="21" fill="1" visible="no" active="no"/>
+<layer number="14" name="Route14" color="22" fill="1" visible="no" active="no"/>
+<layer number="15" name="Route15" color="23" fill="1" visible="no" active="no"/>
+<layer number="16" name="Bottom" color="1" fill="1" visible="no" active="no"/>
+<layer number="17" name="Pads" color="2" fill="1" visible="no" active="no"/>
+<layer number="18" name="Vias" color="2" fill="1" visible="no" active="no"/>
+<layer number="19" name="Unrouted" color="6" fill="1" visible="no" active="no"/>
+<layer number="20" name="Dimension" color="24" fill="1" visible="no" active="no"/>
+<layer number="21" name="tPlace" color="7" fill="1" visible="no" active="no"/>
+<layer number="22" name="bPlace" color="7" fill="1" visible="no" active="no"/>
+<layer number="23" name="tOrigins" color="15" fill="1" visible="no" active="no"/>
+<layer number="24" name="bOrigins" color="15" fill="1" visible="no" active="no"/>
+<layer number="25" name="tNames" color="7" fill="1" visible="no" active="no"/>
+<layer number="26" name="bNames" color="7" fill="1" visible="no" active="no"/>
+<layer number="27" name="tValues" color="7" fill="1" visible="no" active="no"/>
+<layer number="28" name="bValues" color="7" fill="1" visible="no" active="no"/>
 <layer number="29" name="tStop" color="7" fill="3" visible="no" active="no"/>
 <layer number="30" name="bStop" color="7" fill="6" visible="no" active="no"/>
@@
 <layer number="35" name="tGlue" color="7" fill="4" visible="no" active="no"/>
 <layer number="36" name="bGlue" color="7" fill="5" visible="no" active="no"/>
-<layer number="37" name="tTest" color="7" fill="1" visible="yes" active="no"/>
-<layer number="38" name="bTest" color="7" fill="1" visible="yes" active="no"/>
+<layer number="37" name="tTest" color="7" fill="1" visible="no" active="no"/>
+<layer number="38" name="bTest" color="7" fill="1" visible="no" active="no"/>
 <layer number="39" name="tKeepout" color="4" fill="11" visible="no" active="no"/>
 <layer number="40" name="bKeepout" color="1" fill="11" visible="no" active="no"/>
@@
 <layer number="44" name="Drills" color="7" fill="1" visible="no" active="no"/>
 <layer number="45" name="Holes" color="7" fill="1" visible="no" active="no"/>
-<layer number="46" name="Milling" color="3" fill="1" visible="yes" active="no"/>
-<layer number="47" name="Measures" color="7" fill="1" visible="yes" active="no"/>
-<layer number="48" name="Document" color="7" fill="1" visible="yes" active="no"/>
-<layer number="49" name="Reference" color="7" fill="1" visible="yes" active="no"/>
-<layer number="50" name="dxf" color="7" fill="1" visible="yes" active="no"/>
-<layer number="51" name="tDocu" color="7" fill="1" visible="yes" active="no"/>
-<layer number="52" name="bDocu" color="7" fill="1" visible="yes" active="no"/>
-<layer number="53" name="tGND_GNDA" color="7" fill="9" visible="yes" active="no"/>
-<layer number="54" name="bGND_GNDA" color="1" fill="9" visible="yes" active="no"/>
-<layer number="56" name="wert" color="7" fill="1" visible="yes" active="no"/>
-<layer number="57" name="tCAD" color="7" fill="1" visible="yes" active="no"/>
-<layer number="59" name="tCarbon" color="7" fill="1" visible="yes" active="no"/>
-<layer number="60" name="bCarbon" color="7" fill="1" visible="yes" active="no"/>
+<layer number="46" name="Milling" color="3" fill="1" visible="no" active="no"/>
+<layer number="47" name="Measures" color="7" fill="1" visible="no" active="no"/>
+<layer number="48" name="Document" color="7" fill="1" visible="no" active="no"/>
+<layer number="49" name="Reference" color="7" fill="1" visible="no" active="no"/>
+<layer number="50" name="dxf" color="7" fill="1" visible="no" active="no"/>
+<layer number="51" name="tDocu" color="7" fill="1" visible="no" active="no"/>
+<layer number="52" name="bDocu" color="7" fill="1" visible="no" active="no"/>
+<layer number="53" name="tGND_GNDA" color="7" fill="9" visible="no" active="no"/>
+<layer number="54" name="bGND_GNDA" color="1" fill="9" visible="no" active="no"/>
+<layer number="56" name="wert" color="7" fill="1" visible="no" active="no"/>
+<layer number="57" name="tCAD" color="7" fill="1" visible="no" active="no"/>
+<layer number="59" name="tCarbon" color="7" fill="1" visible="no" active="no"/>
+<layer number="60" name="bCarbon" color="7" fill="1" visible="no" active="no"/>
 <layer number="88" name="SimResults" color="9" fill="1" visible="yes" active="yes"/>
 <layer number="89" name="SimProbes" color="9" fill="1" visible="yes" active="yes"/>

Commit message: Upload V1.1
* Use through-hole headers
* Change CS pin for ESP32 coprocessor
* Fix bugs in previous version (Serial breakout pads for ESP32, I²C header pinout)
Parts:
- J1, J10, J11, J12, J2, J3, J4, J5, J6, J7, J8, J9: device ItsyBitsy_Expander_v1.0:GROVE-CONNECTOR-SMD(4+2P-2.0) -> ItsyBitsy_Expander_v1.0:GROVE-CONNECTOR-4PIN
Connections:
- net SCL: now also J4.1, J5.1, J6.1; no longer J4.2, J5.2, J6.2
- net SDA: now also J4.2, J5.2, J6.2; no longer J4.1, J5.1, J6.1
Changed lines of the file:
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@@
 </classes>
 <parts>
-<part name="J1" library="ItsyBitsy_Expander_v1.0" deviceset="GROVE-CONNECTOR-SMD(4+2P-2.0)" device="" value="H4P-SMD-2.0"/>
+<part name="J1" library="ItsyBitsy_Expander_v1.0" deviceset="GROVE-CONNECTOR-4PIN" device="" value="H4P-SMD-2.0"/>
 <part name="U1" library="ItsyBitsy_Expander_v1.0" deviceset="ESP-WROOM-32" device=""/>
 <part name="FRAME1" library="frames" library_urn="urn:adsk.eagle:library:229" deviceset="DINA4_L" device=""/>
@@
 <part name="U$18" library="ItsyBitsy_Expander_v1.0" deviceset="GND" device=""/>
 <part name="U$19" library="ItsyBitsy_Expander_v1.0" deviceset="GND" device=""/>
-<part name="J2" library="ItsyBitsy_Expander_v1.0" deviceset="GROVE-CONNECTOR-SMD(4+2P-2.0)" device="" value="H4P-SMD-2.0"/>
-<part name="J3" library="ItsyBitsy_Expander_v1.0" deviceset="GROVE-CONNECTOR-SMD(4+2P-2.0)" device="" value="H4P-SMD-2.0"/>
-<part name="J4" library="ItsyBitsy_Expander_v1.0" deviceset="GROVE-CONNECTOR-SMD(4+2P-2.0)" device="" value="H4P-SMD-2.0"/>
-<part name="J5" library="ItsyBitsy_Expander_v1.0" deviceset="GROVE-CONNECTOR-SMD(4+2P-2.0)" device="" value="H4P-SMD-2.0"/>
-<part name="J6" library="ItsyBitsy_Expander_v1.0" deviceset="GROVE-CONNECTOR-SMD(4+2P-2.0)" device="" value="H4P-SMD-2.0"/>
-<part name="J7" library="ItsyBitsy_Expander_v1.0" deviceset="GROVE-CONNECTOR-SMD(4+2P-2.0)" device="" value="H4P-SMD-2.0"/>
-<part name="J8" library="ItsyBitsy_Expander_v1.0" deviceset="GROVE-CONNECTOR-SMD(4+2P-2.0)" device="" value="H4P-SMD-2.0"/>
-<part name="J9" library="ItsyBitsy_Expander_v1.0" deviceset="GROVE-CONNECTOR-SMD(4+2P-2.0)" device="" value="H4P-SMD-2.0"/>
-<part name="J10" library="ItsyBitsy_Expander_v1.0" deviceset="GROVE-CONNECTOR-SMD(4+2P-2.0)" device="" value="H4P-SMD-2.0"/>
-<part name="J11" library="ItsyBitsy_Expander_v1.0" deviceset="GROVE-CONNECTOR-SMD(4+2P-2.0)" device="" value="H4P-SMD-2.0"/>
-<part name="J12" library="ItsyBitsy_Expander_v1.0" deviceset="GROVE-CONNECTOR-SMD(4+2P-2.0)" device="" value="H4P-SMD-2.0"/>
+<part name="J2" library="ItsyBitsy_Expander_v1.0" deviceset="GROVE-CONNECTOR-4PIN" device="" value="H4P-SMD-2.0"/>
+<part name="J3" library="ItsyBitsy_Expander_v1.0" deviceset="GROVE-CONNECTOR-4PIN" device="" value="H4P-SMD-2.0"/>
+<part name="J4" library="ItsyBitsy_Expander_v1.0" deviceset="GROVE-CONNECTOR-4PIN" device="" value="H4P-SMD-2.0"/>
+<part name="J5" library="ItsyBitsy_Expander_v1.0" deviceset="GROVE-CONNECTOR-4PIN" device="" value="H4P-SMD-2.0"/>
+<part name="J6" library="ItsyBitsy_Expander_v1.0" deviceset="GROVE-CONNECTOR-4PIN" device="" value="H4P-SMD-2.0"/>
+<part name="J7" library="ItsyBitsy_Expander_v1.0" deviceset="GROVE-CONNECTOR-4PIN" device="" value="H4P-SMD-2.0"/>
+<part name="J8" library="ItsyBitsy_Expander_v1.0" deviceset="GROVE-CONNECTOR-4PIN" device="" value="H4P-SMD-2.0"/>
+<part name="J9" library="ItsyBitsy_Expander_v1.0" deviceset="GROVE-CONNECTOR-4PIN" device="" value="H4P-SMD-2.0"/>
+<part name="J10" library="ItsyBitsy_Expander_v1.0" deviceset="GROVE-CONNECTOR-4PIN" device="" value="H4P-SMD-2.0"/>
+<part name="J11" library="ItsyBitsy_Expander_v1.0" deviceset="GROVE-CONNECTOR-4PIN" device="" value="H4P-SMD-2.0"/>
+<part name="J12" library="ItsyBitsy_Expander_v1.0" deviceset="GROVE-CONNECTOR-4PIN" device="" value="H4P-SMD-2.0"/>
 <part name="U$31" library="ItsyBitsy_Expander_v1.0" deviceset="GND" device=""/>
 <part name="+3V9" library="ItsyBitsy_Expander_v1.0" deviceset="+3V3" device=""/>
@@
 <instance part="J1" gate="G$1" x="99.06" y="63.5" smashed="yes" rot="R270">
 <attribute name="NAME" x="102.87" y="59.69" size="1.27" layer="95" ratio="10" align="center"/>
-<attribute name="VALUE" x="96.52" y="59.69" size="1.27" layer="96" ratio="10" align="center"/>
 </instance>
 <instance part="U1" gate="G$1" x="-82.55" y="59.69" smashed="yes">
@@
 <instance part="J2" gate="G$1" x="99.06" y="43.18" smashed="yes" rot="R270">
 <attribute name="NAME" x="102.87" y="39.37" size="1.27" layer="95" ratio="10" align="center"/>
-<attribute name="VALUE" x="96.52" y="39.37" size="1.27" layer="96" ratio="10" align="center"/>
 </instance>
 <instance part="J3" gate="G$1" x="99.06" y="22.86" smashed="yes" rot="R270">
 <attribute name="NAME" x="102.87" y="19.05" size="1.27" layer="95" ratio="10" align="center"/>
-<attribute name="VALUE" x="96.52" y="19.05" size="1.27" layer="96" ratio="10" align="center"/>
 </instance>
 <instance part="J4" gate="G$1" x="99.06" y="2.54" smashed="yes" rot="R270">
@@
 <net name="SDA" class="0">
 <segment>
-<pinref part="J4" gate="G$1" pin="1"/>
-<wire x1="102.87" y1="7.62" x2="106.68" y2="7.62" width="0.1524" layer="91"/>
-<label x="102.87" y="7.62" size="1.778" layer="95"/>
-</segment>
-<segment>
-<pinref part="J5" gate="G$1" pin="1"/>
-<wire x1="102.87" y1="-12.7" x2="106.68" y2="-12.7" width="0.1524" layer="91"/>
-<label x="102.87" y="-12.7" size="1.778" layer="95"/>
-</segment>
-<segment>
-<pinref part="J6" gate="G$1" pin="1"/>
-<wire x1="102.87" y1="-33.02" x2="106.68" y2="-33.02" width="0.1524" layer="91"/>
-<label x="102.87" y="-33.02" size="1.778" layer="95"/>
-</segment>
-<segment>
 <wire x1="-44.45" y1="-24.13" x2="-63.5" y2="-24.13" width="0.1524" layer="91"/>
 <label x="-54.61" y="-24.13" size="1.524" layer="95"/>
@@
 <pinref part="R7" gate="G$1" pin="2"/>
 </segment>
-</net>
-<net name="SCL" class="0">
-<segment>
-<pinref part="J4" gate="G$1" pin="2"/>
-<wire x1="100.33" y1="7.62" x2="100.33" y2="10.16" width="0.1524" layer="91"/>
-<wire x1="100.33" y1="10.16" x2="106.68" y2="10.16" width="0.1524" layer="91"/>
-<label x="102.87" y="10.16" size="1.778" layer="95"/>
-</segment>
 <segment>
 <pinref part="J6" gate="G$1" pin="2"/>
 <wire x1="100.33" y1="-33.02" x2="100.33" y2="-30.48" width="0.1524" layer="91"/>
 <wire x1="100.33" y1="-30.48" x2="106.68" y2="-30.48" width="0.1524" layer="91"/>
-<label x="102.87" y="-30.48" size="1.778" layer="95"/>
-</segment>
-<segment>
-<pinref part="J5" gate="G$1" pin="2"/>
+<label x="104.14" y="-30.48" size="1.778" layer="95"/>
+</segment>
+<segment>
 <wire x1="100.33" y1="-12.7" x2="100.33" y2="-10.16" width="0.1524" layer="91"/>
 <wire x1="100.33" y1="-10.16" x2="106.68" y2="-10.16" width="0.1524" layer="91"/>
-<label x="102.87" y="-10.16" size="1.778" layer="95"/>
-</segment>
+<label x="104.14" y="-10.16" size="1.778" layer="95"/>
+<pinref part="J5" gate="G$1" pin="2"/>
+</segment>
+<segment>
+<wire x1="100.33" y1="7.62" x2="100.33" y2="10.16" width="0.1524" layer="91"/>
+<wire x1="100.33" y1="10.16" x2="106.68" y2="10.16" width="0.1524" layer="91"/>
+<label x="104.14" y="10.16" size="1.778" layer="95"/>
+<pinref part="J4" gate="G$1" pin="2"/>
+</segment>
+</net>
+<net name="SCL" class="0">
 <segment>
 <wire x1="-44.45" y1="-21.59" x2="-63.5" y2="-21.59" width="0.1524" layer="91"/>
@@
 <pinref part="R6" gate="G$1" pin="2"/>
 </segment>
-</net>
+<segment>
+<pinref part="J6" gate="G$1" pin="1"/>
+<wire x1="102.87" y1="-33.02" x2="106.68" y2="-33.02" width="0.1524" layer="91"/>
+<label x="104.14" y="-33.02" size="1.778" layer="95"/>
+</segment>
+<segment>
+<wire x1="102.87" y1="-12.7" x2="106.68" y2="-12.7" width="0.1524" layer="91"/>
+<label x="104.14" y="-12.7" size="1.778" layer="95"/>
+<pinref part="J5" gate="G$1" pin="1"/>
+</segment>
+<segment>
+<wire x1="102.87" y1="7.62" x2="106.68" y2="7.62" width="0.1524" layer="91"/>
+<label x="104.14" y="7.62" size="1.778" layer="95"/>
+<pinref part="J4" gate="G$1" pin="1"/>
+</segment>
+</net>
